File: Polemo Core/Polemo Core 2/Polemo Core 2.kicad_sch (KiCad schematic)
At the start: 174 parts, among them P1 Header-Male-2.54_2x2, P2 Header-Male-2.54_2x2, Q1 BC847_C2910145, Q2 MMBT5551LT1G, Q3 AO3401A, Q4 AO3401A, Q5 MMBT5551LT1G, U1 ATSAML21G18B-AUT, U10 74LVC1G08GV,125, U11 LT3014BHVES5#TRMPBF, U12 TXU0202DCUR, U13 TLV7031DBVR, U14 TLR341G-GTR, U15 803-87-006-10-001101, U2 XC6209F332MR-G, U3 MC14043BDR2G, U4 LMV793MFX/NOPB, U5 TPS7A2030PDBVR, U6 TLV3201AIDBVT, U7 OPA357AIDBVR, U8 TLR341G-GTR, U9 MF-ASML020/6-2, X1 32.768kHz

Commit message: Moved more components around
Parts:
- C38, C39: footprint Capacitor_SMD:C_0805_2012Metric -> Capacitor_SMD:C_1812_4532Metric
Changed lines of the file:
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@@
 		(lib_id "1206B475K500NT_2")
 		(at 316.23 285.75 0)
-		(unit 0)
+		(unit 1)
 		(exclude_from_sim no)
 		(in_bom yes)
@@
 			)
 		)
-		(property "Footprint" "Capacitor_SMD:C_0805_2012Metric"
+		(property "Footprint" "Capacitor_SMD:C_1812_4532Metric"
 			(at 316.23 285.75 0)
 			(effects
@@
 				(path "/0190368d-9c8f-48e4-a1da-81c8419b9305"
 					(reference "C39")
-					(unit 0)
+					(unit 1)
 				)
 			)
@@
 		(lib_id "1206B475K500NT_3")
 		(at 306.07 285.75 0)
-		(unit 0)
+		(unit 1)
 		(exclude_from_sim no)
 		(in_bom yes)
@@
 			)
 		)
-		(property "Footprint" "Capacitor_SMD:C_0805_2012Metric"
+		(property "Footprint" "Capacitor_SMD:C_1812_4532Metric"
 			(at 306.07 285.75 0)
 			(effects
@@
 				(path "/0190368d-9c8f-48e4-a1da-81c8419b9305"
 					(reference "C38")
-					(unit 0)
+					(unit 1)
 				)
 			)

Commit message: Added source code for the firmw.are
Connections:
- net 3V0: no longer C11.2, C2.2, C3.2
- net 3V3: now also C11.2, C2.2, C3.2, R27.1, U10.4 (Y); no longer MEAS1.2, TP7.1
- net SHAPER_OUT: no longer names the net of H5.3, R17.1, R19.2, TP10.1, U4.1 (OUTPUT), U6.3 (VIN+)
- net SHAPER_OUT: no longer C15.2, R17.2, U7.3 (IN+)
- new net: C15.2, R17.2, U7.3 (IN+)
- new net: MEAS1.2, TP7.1
Other:
- moved on the sheet: BUT1, C1, C10, C11, C12, C13, C14, C15, C16, C17, C18, C19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
