File: Polemo Core/Polemo Core 2/Polemo Core 2.kicad_sch (KiCad schematic)
At the start: 174 parts, among them P1 Header-Male-2.54_2x2, P2 Header-Male-2.54_2x2, Q1 BC847_C2910145, Q2 MMBT5551LT1G, Q3 AO3401A, Q4 AO3401A, Q5 MMBT5551LT1G, U1 ATSAML21G18B-AUT, U10 74LVC1G08GV,125, U11 LT3014BHVES5#TRMPBF, U12 TXU0202DCUR, U13 TLV7031DBVR, U14 TLR341G-GTR, U15 803-87-006-10-001101, U2 XC6209F332MR-G, U3 MC14043BDR2G, U4 LMV793MFX/NOPB, U5 TPS7A2030PDBVR, U6 TLV3201AIDBVT, U7 OPA357AIDBVR, U8 TLR341G-GTR, U9 MF-ASML020/6-2, X1 32.768kHz

Commit message: Added README.md and update many files
Other:
- moved on the sheet: C48, C49, C50, C52, TP16, TP17
